Commit message: camera stl

File: urdf/grabette_right/robot.urdf (robot description, URDF)
Before this commit: robot grabette_right, 3 links, 2 joints
Links:
- added link camera, mass 1e-9
- added link imu, mass 1e-9
- link thumb_base: geometry collision mesh filename=package://grabette_right/assets/b0404.stl; collision mesh filename=package://grabette_right/assets/bmi088.stl
Joints:
- added joint camera_frame: type fixed, parent thumb_base, child camera, origin xyz=-0.0408438 -0.0494999 0.044 rpy=1.5708 -0 3.14159, axis 0 0 0
- added joint imu_frame: type fixed, parent thumb_base, child imu, origin xyz=-0.0408438 -0.0631499 0.044 rpy=1.5708 -0 0, axis 0 0 0
