Commit message: Fix post-processing for upright OAK.

File: packages/grabette/urdf/grabette_right/robot.urdf (robot description, URDF)
Before this commit: robot grabette_right, 5 links, 4 joints
Joints:
- joint camera_frame: origin xyz=-0.0408438 -0.0494999 0.044 rpy=1.5708 -0 3.14159 -> xyz=-0.0408438 -0.0494999 0.044 rpy=1.5708 -0 0

Commit message: updated urdf

File: packages/grabette/urdf/grabette_right/robot.urdf (robot description, URDF)
Before this commit: robot grabette_right, 5 links, 4 joints
Links:
- removed link imu
- removed link phalanx_1_bottom
- removed link phalanx_2
- removed link thumb_base
- added link distal_r, mass 0.0252381; collision mesh filename=package://assets/distal_r.stl; collision mesh filename=package://assets/distal_soft_tip.stl
- added link finger_tip, mass 1e-9
- added link grip_r, mass 0.256238; collision mesh filename=package://assets/602_00009_phillips_flat_head__m2_x_0_40mm_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; collision mesh filename=package://assets/602_00009_phillips_flat_head__m2_x_0_40mm_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
- added link gripper_base, mass 1e-9
- added link gripper_center, mass 1e-9
- added link oak_l, mass 1e-9
- added link oak_r, mass 1e-9
- added link proximal_bend_r, mass 0.0318375; collision mesh filename=package://assets/bushing_6x8x4.stl; collision mesh filename=package://assets/bushing_6x8x4.stl
- added link thumb_tip, mass 1e-9
Joints:
- removed joint imu_frame
- added joint finger_tip_frame: type fixed, parent distal_r, child finger_tip, origin xyz=0.0243384 0.0565209 -0.0232 rpy=-1.5708 -0 0.643367, axis 0 0 0
- added joint gripper_base_frame: type fixed, parent grip_r, child gripper_base, origin xyz=0.0337996 0.055 -0.0232 rpy=1.5708 -0 3.14159, axis 0 0 0
- added joint gripper_center_frame: type fixed, parent grip_r, child gripper_center, origin xyz=0.0373485 -0.0335873 -0.0232 rpy=-0 0 -1.5708, axis 0 0 0
- added joint oak_l_frame: type fixed, parent grip_r, child oak_l, origin xyz=0.0373486 0.025667 0.0298246 rpy=-1.5708 -0 3.14159, axis 0 0 0
- added joint oak_r_frame: type fixed, parent grip_r, child oak_r, origin xyz=0.0173486 0.025667 0.0298246 rpy=-1.5708 -0 3.14159, axis 0 0 0
- added joint thumb_tip_frame: type fixed, parent grip_r, child thumb_tip, origin xyz=0.0910992 -0.0551614 -0.0232 rpy=-1.5708 -0 2.34214, axis 0 0 0
- joint camera_frame: origin xyz=-0.0408438 -0.0494999 0.044 rpy=1.5708 -0 0 -> xyz=0.0408486 0.033623 0.0731261 rpy=-1.91986 0 3.14159; parent thumb_base -> grip_r
- joint distal: child phalanx_2 -> distal_r; limit lower=-3.141592653589793 upper=3.141592653589793 effort=10 velocity=10 -> lower=0 upper=1.5708 effort=10 velocity=10; origin xyz=0.0321391 -0.0383025 -0 rpy=3.14159 -0 0 -> xyz=0.0321391 0.0383025 0 rpy=0 0 0; parent phalanx_1_bottom -> proximal_bend_r
- joint proximal: child phalanx_1_bottom -> grip_r; limit lower=-3.141592653589793 upper=3.141592653589793 effort=10 velocity=10 -> lower=-1.5708 upper=0 effort=10 velocity=10; origin xyz=0 -0 0 rpy=3.14159 -0 -0 -> xyz=-0 0 -0 rpy=-0 -0 -3.14159; parent thumb_base -> proximal_bend_r

File: packages/gripette/urdf/gripette_right/robot.urdf (robot description, URDF)
Before this commit: robot gripette_right, 5 links, 4 joints
Links:
- removed link distal
- removed link feetech_sts3215__configuration_default
- removed link openarm_fix
- added link distal_r, mass 0.0238623; collision mesh filename=package://assets/distal_r.stl; collision mesh filename=package://assets/distal_soft_tip.stl
- added link finger_tip, mass 1e-9
- added link gripper_base_r, mass 0.227294; collision mesh filename=package://assets/602_00009_phillips_flat_head__m2_x_0_40mm_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; collision mesh filename=package://assets/602_00009_phillips_flat_head__m2_x_0_40mm_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
- added link gripper_center, mass 1e-9
- added link oak_l, mass 1e-9
- added link oak_r, mass 1e-9
- added link proximal_bot_r, mass 0.0769363; collision mesh filename=package://assets/cross_bar.stl; collision mesh filename=package://assets/feetech_pt_screw_2x6__configuration_defaul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
- added link thumb_tip, mass 1e-9
- link gripper_base: mass 0.225894 -> 1e-9; geometry 
Joints:
- removed joint openarm_fix_frame
- added joint finger_tip_frame: type fixed, parent distal_r, child finger_tip, origin xyz=-0.0613312 -0.00504543 0.01905 rpy=-1.5708 -0 2.70286, axis 0 0 0
- added joint gripper_base_frame: type fixed, parent gripper_base_r, child gripper_base, origin xyz=-0.0338 -0.055 -0.0232 rpy=1.5708 -0 0, axis 0 0 0
- added joint gripper_center_frame: type fixed, parent gripper_base_r, child gripper_center, origin xyz=-0.0373485 0.0335873 -0.0232 rpy=-0 -0 1.5708, axis 0 0 0
- added joint oak_l_frame: type fixed, parent gripper_base_r, child oak_l, origin xyz=-0.0373486 -0.025667 0.0298246 rpy=-1.5708 -0 0, axis 0 0 0
- added joint oak_r_frame: type fixed, parent gripper_base_r, child oak_r, origin xyz=-0.0173486 -0.025667 0.0298246 rpy=-1.5708 -0 0, axis 0 0 0
- added joint thumb_tip_frame: type fixed, parent gripper_base_r, child thumb_tip, origin xyz=-0.0910992 0.0551614 -0.0232 rpy=-1.5708 0 -0.799448, axis 0 0 0
- joint camera_frame: origin xyz=0.0030569 -0.0657041 0.0938888 rpy=-1.5708 -0 0 -> xyz=-0.0408486 -0.033623 0.0731261 rpy=-1.91986 -0 0; parent gripper_base -> gripper_base_r
- joint distal: child distal -> distal_r; limit lower=-2.0944 upper=0 effort=10 velocity=10 -> lower=-0 upper=1.5708 effort=10 velocity=10; origin xyz=0.0249998 -0.0433013 -0.00055 rpy=0 0 2.0944 -> xyz=-0.0383025 0.0321391 -0.0001 rpy=-0 -0 -0.488692; parent feetech_sts3215__configuration_default -> proximal_bot_r
- joint proximal: child feetech_sts3215__configuration_default -> proximal_bot_r; limit lower=-1.57079 upper=7.64992e-06 effort=10 velocity=10 -> lower=-0 upper=1.5708 effort=10 velocity=10; origin xyz=0.0439007 -0.0248042 0.0428388 rpy=-3.14159 -0 -0.174525 -> xyz=0 0 -0.04225 rpy=0 -0 -1.5708; parent gripper_base -> gripper_base_r

File: packages/gripette/urdf/openarm_gripette_right/robot.urdf (robot description, URDF)
Before this commit: robot openarm_gripette_right, 5 links, 4 joints
Links:
- removed link distal
- removed link openarm_fix
- added link distal_soft_tip, mass 0.0238623; collision mesh filename=package://assets/distal_r.stl; collision mesh filename=package://assets/distal_soft_tip.stl
- added link dm_j4310_1_2_step, mass 1e-09; collision mesh filename=package://assets/dm_j4310_1_2_step.stl; collision mesh filename=package://assets/j4_c_2_step.stl
- added link dm_j4310_1_2_step_2, mass 1e-09; collision mesh filename=package://assets/dm_j4310_1_2_step_2.stl; collision mesh filename=package://assets/fl6700zz_2_step.stl
- added link dm_j4340_2_step, mass 1e-09; collision mesh filename=package://assets/dm_j4340_2_step.stl; collision mesh filename=package://assets/dm_j4340p_2_step.stl
- added link dm_j8009p_2_step_1, mass 1e-09; collision mesh filename=package://assets/dm_j8009p_2_step_1.stl; collision mesh filename=package://assets/j1_c_1_step.stl
- added link finger_tip, mass 1e-9
- added link gripper_center, mass 1e-9
- added link hfsb6_6060_750_1_step, mass 1e-09; collision mesh filename=package://assets/dm_j8009p_2_step.stl; collision mesh filename=package://assets/hfsb6_6060_750_1_step.stl
- added link j2_b_2_step, mass 1e-09; collision mesh filename=package://assets/j2_a_1_step.stl; collision mesh filename=package://assets/j2_b_2_step.stl
- added link j6_a_3_step, mass 1e-09; collision mesh filename=package://assets/dm_j4310_1_2_step_1.stl; collision mesh filename=package://assets/j5_a_3_step.stl
- added link j7_e_2_step, mass 1e-09; collision mesh filename=package://assets/j7_e_2_step.stl; visual mesh filename=package://assets/j7_e_2_step.stl
- added link j8_a_2_step, mass 0.227294; collision mesh filename=package://assets/602_00009_phillips_flat_head__m2_x_0_40mm_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; collision mesh filename=package://assets/602_00009_phillips_flat_head__m2_x_0_40mm_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
- added link oak_l, mass 1e-9
- added link oak_r, mass 1e-9
- added link thumb_tip, mass 1e-9
- link feetech_sts3215__configuration_default: mass 0.101487 -> 0.0769363; geometry collision mesh filename=package://assets/cross_bar.stl; collision mesh filename=package://assets/feetech_pt_screw_2x6__configuration_defaul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
- link gripper_base: mass 0.225894 -> 1e-9; geometry 
Joints:
- removed joint openarm_fix_frame
- added joint finger_tip_frame: type fixed, parent distal_soft_tip, child finger_tip, origin xyz=-0.0613312 -0.00504543 0.01905 rpy=-1.5708 -0 2.70286, axis 0 0 0
- added joint gripper_base_frame: type fixed, parent j8_a_2_step, child gripper_base, origin xyz=-0 0.0495 0.0205 rpy=1.5708 1.5708 0, axis 0 0 0
- added joint gripper_center_frame: type fixed, parent j8_a_2_step, child gripper_center, origin xyz=-0 0.138087 0.0240485 rpy=1.5708 0 1.5708, axis 0 0 0
- added joint oak_l_frame: type fixed, parent j8_a_2_step, child oak_l, origin xyz=0.0530246 0.078833 0.0240486 rpy=-1.5708 1.5708 0, axis 0 0 0
- added joint oak_r_frame: type fixed, parent j8_a_2_step, child oak_r, origin xyz=0.0530246 0.078833 0.00404864 rpy=-1.5708 1.5708 0, axis 0 0 0
- added joint r_arm_pitch: type revolute, parent hfsb6_6060_750_1_step, child dm_j8009p_2_step_1, origin xyz=-0 -0.0925 0.689 rpy=-1.5708 0.00627138 -0, axis 0 0 1, limit lower=-3.00627 upper=0.993715 effort=10 velocity=10
- added joint r_arm_roll: type revolute, parent dm_j8009p_2_step_1, child j2_b_2_step, origin xyz=-0.0301 -0 -0.06 rpy=-1.5708 -1.56864 -1.5708, axis 0 0 1, limit lower=-3.31828 upper=0.172375 effort=10 velocity=10
- added joint r_arm_yaw: type revolute, parent j2_b_2_step, child dm_j4340_2_step, origin xyz=-0 -0.06625 0.0301 rpy=-1.5708 -1.5708 0, axis 0 0 1, limit lower=-1.57017 upper=1.57142 effort=10 velocity=10
- added joint r_elbow: type revolute, parent dm_j4340_2_step, child dm_j4310_1_2_step, origin xyz=-1.97166e-05 -0.03155 -0.15375 rpy=-1.5708 -5.7e-11 -0.000624931, axis 0 0 1, limit lower=-2.44346 upper=5.7e-11 effort=10 velocity=10
- added joint r_wrist_pitch: type revolute, parent dm_j4310_1_2_step_2, child j8_a_2_step, origin xyz=0.0205 -0 -0.0343 rpy=1.5708 -1.54715 -1.5708, axis 0 0 1, limit lower=-1.54715 upper=1.59445 effort=10 velocity=10
- added joint r_wrist_roll: type revolute, parent j6_a_3_step, child j7_e_2_step, origin xyz=0.0171947 -0.000425585 -0.0455 rpy=-1.5708 0.0176931 1.54605, axis 0 0 1, limit lower=-0.803091 upper=0.767705 effort=10 velocity=10
- added joint r_wrist_roll_mimic: type revolute, parent j6_a_3_step, child dm_j4310_1_2_step_2, origin xyz=0.0342895 -0.000848696 -0.1205 rpy=-1.5708 -0.0176931 -1.59554, axis 0 0 1, limit lower=-3.141592653589793 upper=3.141592653589793 effort=10 velocity=10, mimic joint=r_wrist_roll multiplier=-1.0
- added joint r_wrist_yaw: type revolute, parent dm_j4310_1_2_step, child j6_a_3_step, origin xyz=-0 0.0955 0.0315 rpy=1.5708 -0 0, axis 0 0 1, limit lower=-1.54605 upper=1.59554 effort=10 velocity=10
- added joint thumb_tip_frame: type fixed, parent j8_a_2_step, child thumb_tip, origin xyz=-0 0.159661 0.0777992 rpy=3.14159 0.771348 -1.5708, axis 0 0 0
- joint camera_frame: origin xyz=0.0030569 -0.0657041 0.0938888 rpy=-1.5708 -0 0 -> xyz=0.0963261 0.070877 0.0275486 rpy=-1.91986 1.5708 0; parent gripper_base -> j8_a_2_step
- joint distal: child distal -> distal_soft_tip; limit lower=-2.0944 upper=0 effort=10 velocity=10 -> lower=0 upper=1.5708 effort=10 velocity=10; origin xyz=0.0249998 -0.0433013 -0.00055 rpy=0 0 2.0944 -> xyz=-0.0383025 0.0321391 -0.0001 rpy=-0 -0 -0.488692
- joint proximal: limit lower=-1.57079 upper=7.64992e-06 effort=10 velocity=10 -> lower=0 upper=1.5708 effort=10 velocity=10; origin xyz=0.0439007 -0.0248042 0.0428388 rpy=-3.14159 -0 -0.174525 -> xyz=-0.01905 0.1045 -0.0133 rpy=-1.5708 -0 -1.5708; parent gripper_base -> j8_a_2_step
