Commit message: simu

File: integrations/openarm/openarm_gripette_model/openarm_gripette_model/openarm_right/robot.urdf (robot description, URDF)
Before this commit: robot robot, 14 links, 13 joints
Links:
- removed link distal
- removed link gripper
- removed link openarm_fix
- added link distal_soft_tip, mass 0.0238623; collision mesh filename=package://assets/distal_r.stl; collision mesh filename=package://assets/distal_soft_tip.stl
- added link finger_tip, mass 1e-9
- added link gripper_center, mass 1e-9
- added link j8_a_2_step, mass 0.227294; collision mesh filename=package://assets/602_00009_phillips_flat_head__m2_x_0_40mm_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; collision mesh filename=package://assets/602_00009_phillips_flat_head__m2_x_0_40mm_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
- added link oak_l, mass 1e-9
- added link oak_r, mass 1e-9
- added link thumb_tip, mass 1e-9
- link dm_j4310_1_2_step: geometry collision mesh filename=package://assets/dm_j4310_1_2_step.stl; collision mesh filename=package://assets/j4_c_2_step.stl
- link dm_j4310_1_2_step_2: geometry collision mesh filename=package://assets/dm_j4310_1_2_step_2.stl; collision mesh filename=package://assets/fl6700zz_2_step.stl
- link dm_j4340_2_step: geometry collision mesh filename=package://assets/dm_j4340_2_step.stl; collision mesh filename=package://assets/dm_j4340p_2_step.stl
- link dm_j8009p_2_step_1: geometry collision mesh filename=package://assets/dm_j8009p_2_step_1.stl; collision mesh filename=package://assets/j1_c_1_step.stl
- link feetech_sts3215__configuration_default: mass 0.100722 -> 0.0769363; geometry collision mesh filename=package://assets/cross_bar.stl; collision mesh filename=package://assets/feetech_pt_screw_2x6__configuration_defaul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
- link gripper_base: mass 0.208245 -> 1e-9; geometry 
- link hfsb6_6060_750_1_step: geometry collision mesh filename=package://assets/dm_j8009p_2_step.stl; collision mesh filename=package://assets/hfsb6_6060_750_1_step.stl
- link j2_b_2_step: geometry collision mesh filename=package://assets/j2_a_1_step.stl; collision mesh filename=package://assets/j2_b_2_step.stl
- link j6_a_3_step: geometry collision mesh filename=package://assets/dm_j4310_1_2_step_1.stl; collision mesh filename=package://assets/j5_a_3_step.stl
- link j7_e_2_step: geometry collision mesh filename=package://assets/j7_e_2_step.stl; visual mesh filename=package://assets/j7_e_2_step.stl
Joints:
- removed joint gripper_frame
- removed joint openarm_fix_frame
- added joint finger_tip_frame: type fixed, parent distal_soft_tip, child finger_tip, origin xyz=-0.0613312 -0.00504543 0.01905 rpy=-1.5708 -0 2.70286, axis 0 0 0
- added joint gripper_base_frame: type fixed, parent j8_a_2_step, child gripper_base, origin xyz=-0 0.0495 0.0205 rpy=1.5708 1.5708 0, axis 0 0 0
- added joint gripper_center_frame: type fixed, parent j8_a_2_step, child gripper_center, origin xyz=-0 0.138087 0.0240485 rpy=1.5708 0 1.5708, axis 0 0 0
- added joint oak_l_frame: type fixed, parent j8_a_2_step, child oak_l, origin xyz=0.0530246 0.078833 0.0240486 rpy=-1.5708 1.5708 0, axis 0 0 0
- added joint oak_r_frame: type fixed, parent j8_a_2_step, child oak_r, origin xyz=0.0530246 0.078833 0.00404864 rpy=-1.5708 1.5708 0, axis 0 0 0
- added joint thumb_tip_frame: type fixed, parent j8_a_2_step, child thumb_tip, origin xyz=-0 0.159661 0.0777992 rpy=3.14159 0.771348 -1.5708, axis 0 0 0
- joint camera_frame: origin xyz=0.0689844 0.0662 0.0278102 rpy=-1.5708 1.5708 0 -> xyz=0.0963261 0.070877 0.0275486 rpy=-1.91986 1.5708 0; parent gripper_base -> j8_a_2_step
- joint distal: child distal -> distal_soft_tip; limit lower=-2.0944 upper=0 effort=10 velocity=10 -> lower=0 upper=1.5708 effort=10 velocity=10; origin xyz=0.025 -0.0433013 -0.00055 rpy=0 0 2.0944 -> xyz=-0.0383025 0.0321391 -0.0001 rpy=-0 -0 -0.488692
- joint proximal: limit lower=-1.5708 upper=0 effort=10 velocity=10 -> lower=0 upper=1.5708 effort=10 velocity=10; origin xyz=0.0179344 0.1065 -0.0131898 rpy=1.5708 1.39626 -1.5708 -> xyz=-0.01905 0.1045 -0.0133 rpy=-1.5708 -0 -1.5708; parent gripper_base -> j8_a_2_step
- joint r_arm_pitch: limit lower=-1.0301 upper=2.96989 effort=10 velocity=10 -> lower=-3.00627 upper=0.993715 effort=10 velocity=10; origin xyz=-0 -0.0925 0.689 rpy=1.5708 -0.0301087 -0 -> xyz=-0 -0.0925 0.689 rpy=-1.5708 0.00627138 -0
- joint r_arm_roll: limit lower=-0.158726 upper=3.33193 effort=10 velocity=10 -> lower=-3.31828 upper=0.172375 effort=10 velocity=10; origin xyz=-0.0301 0 0.06 rpy=-1.5708 1.55499 1.5708 -> xyz=-0.0301 -0 -0.06 rpy=-1.5708 -1.56864 -1.5708
- joint r_arm_yaw: axis 0 0 -1 -> 0 0 1; limit lower=-1.57405 upper=1.56755 effort=10 velocity=10 -> lower=-1.57017 upper=1.57142 effort=10 velocity=10; origin xyz=-0 0.06625 -0.0301 rpy=1.5708 1.5708 0 -> xyz=-0 -0.06625 0.0301 rpy=-1.5708 -1.5708 0
- joint r_elbow: limit lower=-0 upper=2.44346 effort=10 velocity=10 -> lower=-2.44346 upper=5.7e-11 effort=10 velocity=10; origin xyz=-0.000102553 -0.0315498 -0.15375 rpy=1.5708 -0 -0.00325049 -> xyz=-1.97166e-05 -0.03155 -0.15375 rpy=-1.5708 -5.7e-11 -0.000624931
- joint r_wrist_pitch: axis 0 0 -1 -> 0 0 1; child gripper_base -> j8_a_2_step; limit lower=-1.54592 upper=1.59567 effort=10 velocity=10 -> lower=-1.54715 upper=1.59445 effort=10 velocity=10; origin xyz=0.0205 -0 -0.0343 rpy=-1.5708 -1.54592 1.5708 -> xyz=0.0205 -0 -0.0343 rpy=1.5708 -1.54715 -1.5708
- joint r_wrist_roll: axis 0 0 -1 -> 0 0 1; limit lower=-0.796602 upper=0.774194 effort=10 velocity=10 -> lower=-0.803091 upper=0.767705 effort=10 velocity=10; origin xyz=0.0172 2.81739e-05 -0.0455 rpy=1.5708 0.0112042 1.57243 -> xyz=0.0171947 -0.000425585 -0.0455 rpy=-1.5708 0.0176931 1.54605
- joint r_wrist_roll_mimic: mimic joint=r_wrist_roll_inv multiplier=1.0 -> joint=r_wrist_roll multiplier=-1.0; origin xyz=0.0343 5.61841e-05 -0.1205 rpy=-1.5708 -0.0112042 -1.56916 -> xyz=0.0342895 -0.000848696 -0.1205 rpy=-1.5708 -0.0176931 -1.59554
- joint r_wrist_yaw: axis 0 0 -1 -> 0 0 1; limit lower=-1.56916 upper=1.57243 effort=10 velocity=10 -> lower=-1.54605 upper=1.59554 effort=10 velocity=10; origin xyz=-0 -0.0955 -0.0315 rpy=-1.5708 0 -0 -> xyz=-0 0.0955 0.0315 rpy=1.5708 -0 0

Commit message: models now ok. Need to check sign with real world

File: integrations/openarm/openarm_gripette_model/openarm_gripette_model/openarm_right/robot.urdf (robot description, URDF)
Before this commit: robot openarm_gripette_right, 18 links, 17 joints
Joints:
- joint camera_frame: origin xyz=0.0963261 0.070877 0.0275486 rpy=-1.91986 1.5708 0 -> xyz=0.0933847 -0.0789583 -0.0275486 rpy=1.22173 -1.5708 0
- joint distal: origin xyz=-0.0383025 0.0321391 -0.0001 rpy=-0 -0 -0.488692 -> xyz=-0.0383025 0.0321391 -0.0001 rpy=-0 0 -0.488692
- joint gripper_base_frame: origin xyz=-0 0.0495 0.0205 rpy=1.5708 1.5708 0 -> xyz=-0 -0.0495 -0.0205 rpy=-1.5708 -1.5708 0
- joint gripper_center_frame: origin xyz=-0 0.138087 0.0240485 rpy=1.5708 0 1.5708 -> xyz=-0 -0.138087 -0.0240485 rpy=-1.5708 0 -1.5708
- joint oak_l_frame: origin xyz=0.0530246 0.078833 0.0240486 rpy=-1.5708 1.5708 0 -> xyz=0.0530246 -0.078833 -0.0240486 rpy=1.5708 -1.5708 0
- joint oak_r_frame: origin xyz=0.0530246 0.078833 0.00404864 rpy=-1.5708 1.5708 0 -> xyz=0.0530246 -0.078833 -0.00404864 rpy=1.5708 -1.5708 0
- joint proximal: origin xyz=-0.01905 0.1045 -0.0133 rpy=-1.5708 -0 -1.5708 -> xyz=-0.01905 -0.1045 0.0133 rpy=1.5708 -0 1.5708
- joint r_arm_pitch: limit lower=-3.00627 upper=0.993715 effort=10 velocity=10 -> lower=-1.39626 upper=3.49066 effort=10 velocity=10; origin xyz=-0 -0.0925 0.689 rpy=-1.5708 0.00627138 -0 -> xyz=-0 -0.0925 0.689 rpy=1.5708 0 -0
- joint r_arm_roll: limit lower=-3.31828 upper=0.172375 effort=10 velocity=10 -> lower=-1.74533 upper=1.74533 effort=10 velocity=10; origin xyz=-0.0301 -0 -0.06 rpy=-1.5708 -1.56864 -1.5708 -> xyz=-0.0301 -0 0.06 rpy=-3.14159 1.5708 0
- joint r_arm_yaw: limit lower=-1.57017 upper=1.57142 effort=10 velocity=10 -> lower=-1.5708 upper=1.5708 effort=10 velocity=10; origin xyz=-0 -0.06625 0.0301 rpy=-1.5708 -1.5708 0 -> xyz=-0 0.06625 -0.0301 rpy=-1.5708 1.5708 0
- joint r_elbow: limit lower=-2.44346 upper=5.7e-11 effort=10 velocity=10 -> lower=0 upper=2.44346 effort=10 velocity=10; origin xyz=-1.97166e-05 -0.03155 -0.15375 rpy=-1.5708 -5.7e-11 -0.000624931 -> xyz=0 0.03155 0.15375 rpy=-1.5708 0 0
- joint r_wrist_pitch: limit lower=-1.54715 upper=1.59445 effort=10 velocity=10 -> lower=-1.56452 upper=1.57707 effort=10 velocity=10; origin xyz=0.0205 -0 -0.0343 rpy=1.5708 -1.54715 -1.5708 -> xyz=0.0205 0 -0.0343 rpy=1.5708 -1.56452 1.5708
- joint r_wrist_roll: limit lower=-0.803091 upper=0.767705 effort=10 velocity=10 -> lower=-0.78324 upper=0.787556 effort=10 velocity=10; origin xyz=0.0171947 -0.000425585 -0.0455 rpy=-1.5708 0.0176931 1.54605 -> xyz=0.0172 -0 0.0455 rpy=1.5708 0.00215838 -1.5708
- joint r_wrist_roll_mimic: origin xyz=0.0342895 -0.000848696 -0.1205 rpy=-1.5708 -0.0176931 -1.59554 -> xyz=0.0343 -0 0.1205 rpy=1.5708 -0.00215838 1.5708
- joint r_wrist_yaw: limit lower=-1.54605 upper=1.59554 effort=10 velocity=10 -> lower=-1.5708 upper=1.5708 effort=10 velocity=10; origin xyz=-0 0.0955 0.0315 rpy=1.5708 -0 0 -> xyz=-0 -0.0955 -0.0315 rpy=1.5708 0 -0
- joint thumb_tip_frame: origin xyz=-0 0.159661 0.0777992 rpy=3.14159 0.771348 -1.5708 -> xyz=-0 -0.159661 -0.0777992 rpy=0 -0.771348 1.5708

File: packages/grabette/urdf/grabette_left/robot.urdf (robot description, URDF)
Before this commit: robot grabette_left, 10 links, 9 joints
Links:
- link grip_l: mass 0.255808 -> 0.255807
Joints:
- joint camera_frame: origin xyz=-0.0408486 0.033623 0.0731261 rpy=1.91986 -0 0 -> xyz=0.0408486 -0.0255417 0.0701847 rpy=1.91986 -0 -3.14159
- joint distal: origin xyz=-0.0321391 0.0383025 -0 rpy=-0 -0 -0 -> xyz=0.0321391 0.0383025 -0 rpy=3.14159 -0 -3.14159
- joint gripper_base_frame: origin xyz=-0.0337996 0.055 -0.0232 rpy=1.5708 0 -3.14159 -> xyz=0.0337996 -0.055 -0.0232 rpy=1.5708 -0 -0
- joint gripper_center_frame: origin xyz=-0.0373485 -0.0335873 -0.0232 rpy=0 -0 -1.5708 -> xyz=0.0373485 0.0335873 -0.0232 rpy=-0 -0 1.5708
- joint oak_l_frame: origin xyz=-0.0173486 0.025667 0.0298246 rpy=-1.5708 0 -3.14159 -> xyz=0.0173486 -0.025667 0.0298246 rpy=-1.5708 -0 -0
- joint oak_r_frame: origin xyz=-0.0373486 0.025667 0.0298246 rpy=-1.5708 0 -3.14159 -> xyz=0.0373486 -0.025667 0.0298246 rpy=-1.5708 -0 -0
- joint proximal: child grip_l -> proximal_bend_l; origin xyz=-0 0 -0 rpy=0 0 3.14159 -> xyz=-0 0 -0 rpy=-3.14159 0 3.14159; parent proximal_bend_l -> grip_l
- joint thumb_tip_frame: origin xyz=-0.0910992 -0.0551614 -0.0232 rpy=-1.5708 0 -2.34214 -> xyz=0.0910992 0.0551614 -0.0232 rpy=-1.5708 0 0.799448

File: packages/grabette/urdf/grabette_right/robot.urdf (robot description, URDF)
Before this commit: robot grabette_right, 10 links, 9 joints
Joints:
- joint camera_frame: origin xyz=0.0408486 0.033623 0.0731261 rpy=-1.91986 0 3.14159 -> xyz=-0.0408486 -0.0255417 0.0701847 rpy=-1.91986 0 0
- joint distal: origin xyz=0.0321391 0.0383025 0 rpy=0 0 0 -> xyz=-0.0321391 0.0383025 0 rpy=-3.14159 -0 3.14159
- joint finger_tip_frame: origin xyz=0.0243384 0.0565209 -0.0232 rpy=-1.5708 -0 0.643367 -> xyz=0.0243384 0.0565209 -0.0232 rpy=-1.5708 0 0.643367
- joint gripper_base_frame: origin xyz=0.0337996 0.055 -0.0232 rpy=1.5708 -0 3.14159 -> xyz=-0.0337996 -0.055 -0.0232 rpy=1.5708 -0 0
- joint gripper_center_frame: origin xyz=0.0373485 -0.0335873 -0.0232 rpy=-0 0 -1.5708 -> xyz=-0.0373485 0.0335873 -0.0232 rpy=0 -0 1.5708
- joint oak_l_frame: origin xyz=0.0373486 0.025667 0.0298246 rpy=-1.5708 -0 3.14159 -> xyz=-0.0373486 -0.025667 0.0298246 rpy=-1.5708 0 0
- joint oak_r_frame: origin xyz=0.0173486 0.025667 0.0298246 rpy=-1.5708 -0 3.14159 -> xyz=-0.0173486 -0.025667 0.0298246 rpy=-1.5708 0 0
- joint proximal: child grip_r -> proximal_bend_r; origin xyz=-0 0 -0 rpy=-0 -0 -3.14159 -> xyz=0 -0 -0 rpy=3.14159 0 3.14159; parent proximal_bend_r -> grip_r
- joint thumb_tip_frame: origin xyz=0.0910992 -0.0551614 -0.0232 rpy=-1.5708 -0 2.34214 -> xyz=-0.0910992 0.0551614 -0.0232 rpy=-1.5708 -0 -0.799448

File: packages/gripette/urdf/gripette_left/robot.urdf (robot description, URDF)
Before this commit: robot gripette_left, 10 links, 9 joints
Links:
- link gripper_base_l: geometry collision mesh filename=package://assets/602_00009_phillips_flat_head__m2_x_0_40mm_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; collision mesh filename=package://assets/602_00009_phillips_flat_head__m2_x_0_40mm_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
Joints:
- joint camera_frame: origin xyz=0.0408486 -0.033623 0.0731261 rpy=-1.91986 -0 -0 -> xyz=0.0408486 -0.0255417 0.0701847 rpy=-1.91986 -0 -0

File: packages/gripette/urdf/gripette_right/robot.urdf (robot description, URDF)
Before this commit: robot gripette_right, 10 links, 9 joints
Joints:
- joint camera_frame: origin xyz=-0.0408486 -0.033623 0.0731261 rpy=-1.91986 -0 0 -> xyz=-0.0408486 -0.0255417 0.0701847 rpy=-1.91986 -0 0
- joint proximal: limit lower=-0 upper=1.5708 effort=10 velocity=10 -> lower=0 upper=1.5708 effort=10 velocity=10
