Commit message: fix left grabette urdf

File: packages/grabette/urdf/grabette_left/robot.urdf (robot description, URDF)
Before this commit: robot grabette_left, 10 links, 9 joints
Joints:
- joint camera_frame: origin xyz=0.0408486 -0.0255417 0.0701847 rpy=1.91986 -0 -3.14159 -> xyz=0.0408486 -0.0255417 0.0701847 rpy=-1.91986 0 0
